File: UINIO-Signal-Translator.kicad_pcb (KiCad board)
At the start: 2 copper layers, 0 parts

Commit message: Release UINIO-Signal-Translator version 1.0.0.
Parts:
- added C1: 0.1uF, Capacitor_SMD:C_0603_1608Metric, F.Cu at (131.1, 110.4)
- added C2: 0.1uF, Capacitor_SMD:C_0603_1608Metric, F.Cu at (131.1, 102.2)
- added D1: LED Blue, LED_SMD:LED_0603_1608Metric, F.Cu at (136.9, 110.4)
- added D2: LED Blue, LED_SMD:LED_0603_1608Metric, F.Cu at (136.9, 102.2)
- added HOLE**: Hole-1mm, Uinio:Hole-1mm, F.Cu at (125.4, 99.2)
- added HOLE**: Hole-1mm, Uinio:Hole-1mm, F.Cu at (125.4, 113.5)
- added HOLE**: Hole-1mm, Uinio:Hole-1mm, F.Cu at (177.0, 113.5)
- added HOLE**: Hole-1mm, Uinio:Hole-1mm, F.Cu at (177.0, 99.2)
- added J1: Conn_01x02_Pin, Connector_PinHeader_2.54mm:PinHeader_1x02_P2.54mm_Vertical, F.Cu at (127.0, 119.0)
- added J2: Conn_01x08_Pin, Connector_PinHeader_2.54mm:PinHeader_1x08_P2.54mm_Vertical, F.Cu at (137.1, 119.0)
- added J3: Conn_01x02_Pin, Connector_PinHeader_2.54mm:PinHeader_1x02_P2.54mm_Vertical, F.Cu at (127.0, 93.6)
- added J4: Conn_01x08_Pin, Connector_PinHeader_2.54mm:PinHeader_1x08_P2.54mm_Vertical, F.Cu at (137.1, 93.6)
- added J5: Conn_01x08_Pin, Connector_PinHeader_2.54mm:PinHeader_1x08_P2.54mm_Vertical, F.Cu at (157.5, 119.0)
- added J6: Conn_01x03_Pin, Connector_PinHeader_2.54mm:PinHeader_1x03_P2.54mm_Vertical, F.Cu at (156.2, 103.8)
- added J7: Conn_01x08_Pin, Connector_PinHeader_2.54mm:PinHeader_1x08_P2.54mm_Vertical, F.Cu at (157.5, 93.6)
- added R1: 2K, Resistor_SMD:R_0603_1608Metric, F.Cu at (134.0, 110.4)
- added R2: 2K, Resistor_SMD:R_0603_1608Metric, F.Cu at (134.0, 102.2)
- added R3: 10K, Resistor_SMD:R_0603_1608Metric, F.Cu at (156.2, 100.5)
- added U1: TXB0108, Package_SO:TSSOP-20_4.4x6.5mm_P0.65mm, F.Cu at (146.0, 106.3)
- added U2: TXB0108, Package_SO:TSSOP-20_4.4x6.5mm_P0.65mm, F.Cu at (166.4, 106.3)
Routing:
- net /VCCB: track 0.00 -> 51.1 mm, vias 0 -> 3
- net /VCCA: track 0.00 -> 49.8 mm, vias 0 -> 3
- net /OE: track 0.00 -> 25.2 mm
- net GND: track 0.00 -> 18.4 mm, vias 0 -> 7
- net Net-(J7-Pin_8): track 0.00 -> 12.6 mm
- net Net-(J5-Pin_8): track 0.00 -> 12.6 mm
- net Net-(J4-Pin_8): track 0.00 -> 12.6 mm
- net Net-(J2-Pin_8): track 0.00 -> 12.6 mm
- net Net-(J7-Pin_1): track 0.00 -> 12.3 mm
- net Net-(J4-Pin_1): track 0.00 -> 12.3 mm
- net Net-(J5-Pin_1): track 0.00 -> 12.3 mm
- net Net-(J2-Pin_1): track 0.00 -> 12.3 mm
- net Net-(J7-Pin_7): track 0.00 -> 11.8 mm
- net Net-(J5-Pin_7): track 0.00 -> 11.8 mm
- net Net-(J4-Pin_7): track 0.00 -> 11.8 mm
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- added copper zone on B.Cu, net GND
- added copper zone on F.Cu, net GND
Other:
- board outline added: 55.3 x 28.1 mm
- board text added: "A1"
- board text added: "A2"
- board text added: "A3"
- board text added: "A4"
- board text added: "A5"
- board text added: "A6"
- board text added: "A7"
- board text added: "A8"
- board text added: "B1"
- board text added: "B2"
- board text added: "B3"
- board text added: "B4"
- board text added: "B5"
- board text added: "B6"
- board text added: "B7"
- board text added: "B8"
- board text added: "GND"
- board text added: "OE"
- board text added: "TXB0108"
- board text added: "TXB0108 输入电压 1.2V ~ 3.6V 输出电压 1.65V ~ 5.5V"
- board text added: "TXS0108"
- board text added: "TXS0108 输入电压 1.4V ~ 3.6V 输出电压 1.65V ~ 5.5V"
- board text added: "UINIO Signal Translator"
- board text added: "UINIO-Signal-Translator"
- board text added: "UinIO.com"
- board text added: "VCCA"
- board text added: "VCCB"
- board text added: "Version 1.0.0"
- board text added: "➡"
- board text added: "参考电压A"
- board text added: "参考电压B"
- board text added: "电平转换"
- board text added: "输出使能"

Commit message: Release UINIO-Signal-Translator version 2.0.0.
Other:
- board text added: "Version 2.0.0"
- board text removed: "Version 1.0.0"
