File: UINIO-Signal-Translator.kicad_sch (KiCad schematic)
At the start: 0 parts

Commit message: Initialization project.
Other:
- company: 电子技术博客 UinIO.com -> UinIO.com 电子技术实验室
- title: UINIO-Level-Translator -> UINIO-Signal-Translator
Changed lines of the file:
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@@
   (paper "A4")
   (title_block
-    (title "UINIO-Level-Translator")
-    (date "2023-12-29")
+    (title "UINIO-Signal-Translator")
+    (date "2024-01-08")
     (rev "Version 1.0.0")
-    (company "电子技术博客 UinIO.com")
+    (company "UinIO.com 电子技术实验室")
   )
   (sheet_instances

Commit message: Attach more datasheets.
Parts:
- added J1, J3: Conn_01x08_Pin, symbol Connector:Conn_01x08_Pin
- added U1: TXS0108EPW, Package_SO:TSSOP-20_4.4x6.5mm_P0.65mm, symbol Logic_LevelTranslator:TXS0108EPW
Connections:
- new net: J3.1 (Pin_1), U1.1 (A1)
- new net: J3.2 (Pin_2), U1.3 (A2)
- new net: J3.3 (Pin_3), U1.4 (A3)
- new net: J3.4 (Pin_4), U1.5 (A4)
- new net: J3.5 (Pin_5), U1.6 (A5)
- new net: J3.6 (Pin_6), U1.7 (A6)
- new net: J3.7 (Pin_7), U1.8 (A7)
- new net: J3.8 (Pin_8), U1.9 (A8)
- new net: J1.8 (Pin_8), U1.12 (B8)
- new net: J1.7 (Pin_7), U1.13 (B7)
- new net: J1.6 (Pin_6), U1.14 (B6)
- new net: J1.5 (Pin_5), U1.15 (B5)
- new net: J1.4 (Pin_4), U1.16 (B4)
- new net: J1.3 (Pin_3), U1.17 (B3)
- new net: J1.2 (Pin_2), U1.18 (B2)
- new net: J1.1 (Pin_1), U1.20 (B1)
- new net GND: U1.11 (GND)
- new net TXS0108-OE: U1.10 (OE)
- new net TXS0108-VCCA: U1.2 (VCCA)
- new net TXS0108-VCCB: U1.19 (VCCB)
Changed lines of the file:
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@@
 (kicad_sch (version 20230121) (generator eeschema)
-  (paper "A4")
+  (paper "A5")
   (title_block
     (title "UINIO-Signal-Translator")
@@
     (company "UinIO.com 电子技术实验室")
   )
+  (wire (pts (xy 113.665 48.26) (xy 137.16 48.26))
+    (stroke (width 0) (type default))
+  )
+  (wire (pts (xy 68.58 53.34) (xy 93.345 53.34))
+    (stroke (width 0) (type default))
+  )
+  (wire (pts (xy 68.58 48.26) (xy 93.345 48.26))
+    (stroke (width 0) (type default))
+  )
+  (wire (pts (xy 113.665 35.56) (xy 137.16 35.56))
+    (stroke (width 0) (type default))
+  )
+  (wire (pts (xy 113.665 53.34) (xy 137.16 53.34))
+    (stroke (width 0) (type default))
+  )
+  (wire (pts (xy 113.665 43.18) (xy 137.16 43.18))
+    (stroke (width 0) (type default))
+  )
+  (wire (pts (xy 113.665 38.1) (xy 137.16 38.1))
+    (stroke (width 0) (type default))
+  )
+  (wire (pts (xy 120.015 25.4) (xy 106.045 25.4))
+    (stroke (width 0) (type default))
+  )
+  (wire (pts (xy 68.58 45.72) (xy 93.345 45.72))
+    (stroke (width 0) (type default))
+  )
+  (wire (pts (xy 68.58 40.64) (xy 93.345 40.64))
+    (stroke (width 0) (type default))
+  )
+  (wire (pts (xy 113.665 50.8) (xy 137.16 50.8))
+    (stroke (width 0) (type default))
+  )
+  (wire (pts (xy 68.58 35.56) (xy 93.345 35.56))
+    (stroke (width 0) (type default))
+  )
+  (wire (pts (xy 113.665 40.64) (xy 137.16 40.64))
+    (stroke (width 0) (type default))
+  )
+  (wire (pts (xy 115.57 60.96) (xy 103.505 60.96))
+    (stroke (width 0) (type default))
+  )
+  (wire (pts (xy 68.58 50.8) (xy 93.345 50.8))
+    (stroke (width 0) (type default))
+  )
+  (wire (pts (xy 86.995 33.02) (xy 93.345 33.02))
+    (stroke (width 0) (type default))
+  )
+  (wire (pts (xy 86.995 25.4) (xy 100.965 25.4))
+    (stroke (width 0) (type default))
+  )
+  (wire (pts (xy 113.665 45.72) (xy 137.16 45.72))
+    (stroke (width 0) (type default))
+  )
+  (wire (pts (xy 68.58 38.1) (xy 93.345 38.1))
+    (stroke (width 0) (type default))
+  )
+  (wire (pts (xy 68.58 43.18) (xy 93.345 43.18))
+    (stroke (width 0) (type default))
+  )
+  (label "TXS0108-OE" (at 86.995 33.02 180) (fields_autoplaced)
+    (effects (font (size 1.27 1.27)) (justify right bottom))
+  )
+  (label "TXS0108-VCCB" (at 120.015 25.4 0) (fields_autoplaced)
+    (effects (font (size 1.27 1.27)) (justify left bottom))
+  )
+  (label "TXS0108-VCCA" (at 86.995 25.4 180) (fields_autoplaced)
+    (effects (font (size 1.27 1.27)) (justify right bottom))
+  )
+  (symbol (lib_id "Connector:Conn_01x08_Pin") (at 63.5 43.18 0) (unit 1)
+    (in_bom yes) (on_board yes) (dnp no)
+    (property "Reference" "J3" (at 66.04 31.75 0)
+      (effects (font (size 1.27 1.27)))
+    )
+    (property "Value" "Conn_01x08_Pin" (at 66.04 56.515 0)
+      (effects (font (size 1.27 1.27)))
+    )
+    (property "Footprint" "" (at 63.5 43.18 0)
+      (effects (font (size 1.27 1.27)) hide)
+    )
+    (property "Datasheet" "~" (at 63.5 43.18 0)
+      (effects (font (size 1.27 1.27)) hide)
+    )
+    (pin "2")
+    (pin "4")
+    (pin "1")
+    (pin "6")
+    (pin "5")
+    (pin "8")
+    (pin "3")
+    (pin "7")
+    (instances
+      (project "UINIO-Signal-Translator"
+        (path "/c9420995-43a7-497c-95f3-f431f6cd9989"
+          (reference "J3") (unit 1)
+        )
+      )
+    )
+  )
+  (symbol (lib_id "Logic_LevelTranslator:TXS0108EPW") (at 103.505 43.18 0) (unit 1)
+    (in_bom yes) (on_board yes) (dnp no)
+    (property "Reference" "U1" (at 102.235 22.225 0)
+      (effects (font (size 1.27 1.27)) (justify left))
+    )
+    (property "Value" "TXS0108EPW" (at 80.645 60.325 0)
+      (effects (font (size 1.27 1.27)) (justify left))
+    )
+    (property "Footprint" "Package_SO:TSSOP-20_4.4x6.5mm_P0.65mm" (at 103.505 62.23 0)
+      (effects (font (size 1.27 1.27)) hide)
+    )
+    (property "Datasheet" "www.ti.com/lit/ds/symlink/txs0108e.pdf" (at 103.505 45.72 0)
+      (effects (font (size 1.27 1.27)) hide)
+    )
+    (pin "3")
+    (pin "1")
+    (pin "19")
+    (pin "4")
+    (pin "9")
+    (pin "5")
+    (pin "6")
+    (pin "12")
+    (pin "15")
+    (pin "20")
+    (pin "18")
+    (pin "13")
+    (pin "17")
+    (pin "8")
+    (pin "14")
+    (pin "16")
+    (pin "7")
+    (pin "11")
+    (pin "10")
+    (pin "2")
+    (instances
+      (project "UINIO-Signal-Translator"
+        (path "/c9420995-43a7-497c-95f3-f431f6cd9989"
+          (reference "U1") (unit 1)
+        )
+      )
+    )
+  )
+  (symbol (lib_id "Connector:Conn_01x08_Pin") (at 142.24 43.18 0) (mirror y) (unit 1)
+    (in_bom yes) (on_board yes) (dnp no)
+    (property "Reference" "J1" (at 139.7 31.75 0)
+      (effects (font (size 1.27 1.27)))
+    )
+    (property "Value" "Conn_01x08_Pin" (at 140.335 56.515 0)
+      (effects (font (size 1.27 1.27)))
+    )
+    (property "Footprint" "" (at 142.24 43.18 0)
+      (effects (font (size 1.27 1.27)) hide)
+    )
+    (property "Datasheet" "~" (at 142.24 43.18 0)
+      (effects (font (size 1.27 1.27)) hide)
+    )
+    (pin "2")
+    (pin "4")
+    (pin "1")
+    (pin "6")
+    (pin "5")
+    (pin "8")
+    (pin "3")
+    (pin "7")
+    (instances
+      (project "UINIO-Signal-Translator"
+        (path "/c9420995-43a7-497c-95f3-f431f6cd9989"
+          (reference "J1") (unit 1)
+        )
+      )
+    )
+  )
+  (symbol (lib_id "power:GND") (at 115.57 60.96 90) (unit 1)
+    (in_bom yes) (on_board yes) (dnp no)
+    (property "Reference" "#PWR01" (at 121.92 60.96 0)
+      (effects (font (size 1.27 1.27)) hide)
+    )
+    (property "Value" "GND" (at 118.745 60.96 90)
+      (effects (font (size 1.27 1.27)) (justify right))
+    )
+    (property "Footprint" "" (at 115.57 60.96 0)
+      (effects (font (size 1.27 1.27)) hide)
+    )
+    (property "Datasheet" "" (at 115.57 60.96 0)
+      (effects (font (size 1.27 1.27)) hide)
+    )
+    (pin "1")
+    (instances
+      (project "UINIO-Signal-Translator"
+        (path "/c9420995-43a7-497c-95f3-f431f6cd9989"
+          (reference "#PWR01") (unit 1)
+        )
+      )
+    )
+  )
   (sheet_instances

Commit message: Release UINIO-Signal-Translator version 1.0.0.
Parts:
- removed J1, J3: Conn_01x08_Pin, symbol Connector:Conn_01x08_Pin
- added C? (x2): 0.1uF, Capacitor_SMD:C_0603_1608Metric, symbol Device:C
- added D1, D2: LED Blue, LED_SMD:LED_0603_1608Metric, symbol Device:LED
- added J1, J3: Conn_01x02_Pin, Connector_PinHeader_2.54mm:PinHeader_1x02_P2.54mm_Vertical, symbol Connector:Conn_01x02_Pin
- added J2, J4, J5, J7: Conn_01x08_Pin, Connector_PinHeader_2.54mm:PinHeader_1x08_P2.54mm_Vertical, symbol Connector:Conn_01x08_Pin
- added J6: Conn_01x03_Pin, Connector_PinHeader_2.54mm:PinHeader_1x03_P2.54mm_Vertical, symbol Connector:Conn_01x03_Pin
- added R1, R2: 2K, Resistor_SMD:R_0603_1608Metric, symbol Device:R
- added R3: 10K, Resistor_SMD:R_0603_1608Metric, symbol Device:R
- added U2: TXB0108, Package_SO:TSSOP-20_4.4x6.5mm_P0.65mm, symbol Logic_LevelTranslator:TXS0108EPW
- U1: value TXS0108EPW -> TXB0108
Connections:
- net GND: now also C?.1, C?.1, D1.1 (K), D2.1 (K), J1.1 (Pin_1), J3.1 (Pin_1), R3.1, U2.11 (GND)
- net at U1.1 (A1): now also J2.1 (Pin_1)
- net at U1.3 (A2): now also J2.2 (Pin_2)
- net at U1.4 (A3): now also J2.3 (Pin_3)
- net at U1.5 (A4): now also J2.4 (Pin_4)
- net at U1.6 (A5): now also J2.5 (Pin_5)
- net at U1.7 (A6): now also J2.6 (Pin_6)
- net at U1.8 (A7): now also J2.7 (Pin_7)
- net at U1.9 (A8): now also J2.8 (Pin_8)
- net at U1.12 (B8): now also J4.8 (Pin_8)
- net at U1.13 (B7): now also J4.7 (Pin_7)
- net at U1.14 (B6): now also J4.6 (Pin_6)
- net at U1.15 (B5): now also J4.5 (Pin_5)
- net at U1.16 (B4): now also J4.4 (Pin_4)
- net at U1.17 (B3): now also J4.3 (Pin_3)
- net at U1.18 (B2): now also J4.2 (Pin_2)
- net at U1.20 (B1): now also J4.1 (Pin_1)
- net TXS0108-OE renamed OE
- net OE: now also J6.2 (Pin_2), U2.10 (OE)
- net TXS0108-VCCA renamed VCCA
- net VCCA: now also C?.2, J1.2 (Pin_2), J6.3 (Pin_3), R1.1, U2.2 (VCCA)
- net TXS0108-VCCB renamed VCCB
- net VCCB: now also C?.2, J3.2 (Pin_2), R2.1, U2.19 (VCCB)
- new net: J5.1 (Pin_1), U2.1 (A1)
- new net: J7.8 (Pin_8), U2.12 (B8)
- new net: J7.7 (Pin_7), U2.13 (B7)
- new net: J7.6 (Pin_6), U2.14 (B6)
- new net: J7.5 (Pin_5), U2.15 (B5)
- new net: J7.4 (Pin_4), U2.16 (B4)
- new net: J7.3 (Pin_3), U2.17 (B3)
- new net: J7.2 (Pin_2), U2.18 (B2)
- new net: J7.1 (Pin_1), U2.20 (B1)
- new net: J5.2 (Pin_2), U2.3 (A2)
- new net: J5.3 (Pin_3), U2.4 (A3)
- new net: J5.4 (Pin_4), U2.5 (A4)
- new net: J5.5 (Pin_5), U2.6 (A5)
- new net: J5.6 (Pin_6), U2.7 (A6)
- new net: J5.7 (Pin_7), U2.8 (A7)
- new net: J5.8 (Pin_8), U2.9 (A8)
- new net: D1.2 (A), R1.2
- new net: D2.2 (A), R2.2
- new net: J6.1 (Pin_1), R3.2
Other:
- note added: "同时兼容德州仪器 TSSOP20 封装的 TXB0108 与 TXS0108 两款逻辑电平转换芯片"
- moved on the sheet: U1
